Commit message: Implementacao da simulacao e plugin diff_drive do gazebo

File: description/robot.urdf.xacro (robot description, xacro)
@@ -2,3 +2,4 @@
 <robot xmlns:xacro="http://www.ros.org/wiki/xacro"  name="robot">
     <xacro:include filename="robot_core.xacro"/>
+    <xacro:include filename="gazebo_control.xacro"/>
 </robot>

File: description/robot_core.xacro (robot description, xacro)
@@ -40,4 +40,9 @@
         </xacro:inertial_box>
     </link>
+    <gazebo reference="chassis">
+        <material>
+            Gazebo/White
+        </material>
+    </gazebo>
     <!--LEFT WHEEL LINK-->
     <joint name="left_wheel_joint" type="continuous">
@@ -65,4 +70,9 @@
         </xacro:inertial_cylinder>
     </link>
+    <gazebo reference="left_wheel_link">
+        <material>
+            Gazebo/Blue
+        </material>
+    </gazebo>
     <!--RIGHT WHEEL LINK-->
     <joint name="right_wheel_joint" type="continuous">
@@ -90,4 +100,9 @@
         </xacro:inertial_cylinder>
     </link>
+    <gazebo reference="right_wheel_link">
+        <material>
+            Gazebo/Blue
+        </material>
+    </gazebo>
     <!--CASTER WHEEL LINK-->
     <joint name="caster_wheel_link" type="fixed">
@@ -112,3 +127,10 @@
         </xacro:inertial_sphere>
     </link>
+    <gazebo reference="caster_wheel_link">
+        <material>
+            Gazebo/Black
+        </material>
+        <mu1 value="0.001"></mu1>
+        <mu2 value="0.002"></mu2>
+    </gazebo>
 </robot>
